File: PCB/.75-keyboard-PCB.kicad_pcb (KiCad board)
At the start: 2 copper layers, 177 parts, among them J1 SW_Push_45deg, K1 SW_Push_45deg, M1 SW_Push_45deg, P1 SW_Push_45deg, Q1 SW_Push_45deg, T1 SW_Push_45deg, U1 SW_Push_45deg, X1 SW_Push_45deg, Y1 SW_Push_45deg

Commit message: pcb routing finished
Parts:
- removed A1: RaspberryPi_Pico, Module:RaspberryPi_Pico_Common_Unspecified
- removed H1, H2, H3, H4, H5, H6, H7, H8: MountingHole, MountingHole:MountingHole_3.2mm_M3
- added J2: Conn_01x20_Pin, Connector_PinSocket_2.54mm:PinSocket_1x20_P2.54mm_Vertical, B.Cu at (55.2, 108.5)
- added J3: Conn_01x20_Pin, Connector_PinSocket_2.54mm:PinSocket_1x20_P2.54mm_Vertical, B.Cu at (55.2, 90.8)
- moved D60 7.97 mm to (356.2, 136.8)
- moved D58 3.43 mm to (356.2, 146.6)
- moved D59 0.97 mm to (356.2, 124.0)
Routing:
- net GND: track 0.00 -> 382.9 mm
- net EC11B: track 0.00 -> 285.4 mm
- net EC11A: track 0.00 -> 284.6 mm
- net Col14: track 61.9 -> 319.4 mm
- net Col13: track 118.9 -> 343.2 mm
- net Col12: track 115.8 -> 314.9 mm
- net Col11: track 114.4 -> 297.0 mm
- net Col10: track 114.5 -> 280.7 mm
- net Col9: track 113.1 -> 267.6 mm, vias 0 -> 1
- net Col8: track 113.8 -> 249.5 mm, vias 0 -> 1
- net Col7: track 86.5 -> 206.6 mm, vias 0 -> 1
- net Col6: track 87.2 -> 193.9 mm, vias 0 -> 1
- net Col5: track 107.8 -> 194.1 mm, vias 0 -> 1
- net Row5: track 281.1 -> 366.1 mm
- net Col4: track 89.4 -> 165.0 mm, vias 0 -> 1
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Other:
- board outline added: 313.1 x 119 mm

Commit message: kicad switch models
Parts:
- '1, ,1, -1, .1, /1, ;1, <1, =1, >1, A2, Alt2, B1, C1, Ctrl2, D30, Del1, E1, End1, Esc1, F1, F10, F11, F12, F13, F2, F3, F4, F5, F6, F7, F8, F9, Fn1, G1, H9, Home1, I1, Insert1, J1, K1, L1, M1, N10, O1, P1, PgDn1, PgUp1, Q1, R1, S1, T1, U1, V1, V2, W1, X1, Y1, Z1, [1, ]1, ^1, n0, n1, n2, n3, n4, n5, n6, n7, n8, n9, ~1: footprint Button_Switch_Keyboard:SW_Cherry_MX_1.00u_PCB -> Library:3DSW_Cherry_MX_1.00u_PCB
- Alt1, Ctrl1, Win1: footprint Button_Switch_Keyboard:SW_Cherry_MX_1.25u_PCB -> Library:3DSW_Cherry_MX_1.25u_PCB
- Backspace1: footprint Button_Switch_Keyboard:SW_Cherry_MX_2.00u_PCB -> Library:3DSW_Cherry_MX_2.00u_PCB
- Caps1, Shift2: footprint Button_Switch_Keyboard:SW_Cherry_MX_1.75u_PCB -> Library:3D_SW_Cherry_MX_1.75u_PCB
- Enter1, Shift1: footprint Button_Switch_Keyboard:SW_Cherry_MX_2.25u_PCB -> Library:3DSW_Cherry_MX_2.25u_PCB
- Space1: footprint Button_Switch_Keyboard:SW_Cherry_MX_6.25u_PCB -> Library:3DSW_Cherry_MX_6.25u_PCB
- Tab1, \1: footprint Button_Switch_Keyboard:SW_Cherry_MX_1.50u_PCB -> Library:3DSW_Cherry_MX_1.50u_PCB
- moved D87 0.96 mm to (356.2, 161.9)
- moved D88 0.96 mm to (356.2, 180.7)
Routing:
- net Row5: track 366.1 -> 365.2 mm
- net Net-(D88-A): track 13.3 -> 12.3 mm
- net Net-(D87-A): track 13.2 -> 12.2 mm
- net Row4: track 321.4 -> 320.4 mm
Other:
- board size 313.1 x 119 mm -> 309.3 x 118.6 mm
