File: PCB/.75-keyboard-PCB.kicad_pcb (KiCad board)
At the start: 2 copper layers, 309.3 x 118.6 mm, 170 parts, among them J1 SW_Push_45deg, J2 Conn_01x20_Pin, J3 Conn_01x20_Pin, K1 SW_Push_45deg, M1 SW_Push_45deg, P1 SW_Push_45deg, Q1 SW_Push_45deg, T1 SW_Push_45deg, U1 SW_Push_45deg, X1 SW_Push_45deg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

Commit message: idk
Parts:
- moved D87 20.9 mm to (341.4, 147.3), turned to 0 degrees
- moved D15 19.3 mm to (345.9, 90.3)
- moved D59 18.8 mm to (344.6, 109.2), turned to 0 degrees
- moved D58 18.6 mm to (354.0, 128.2), turned to 180 degrees
- moved D88 18.4 mm to (344.6, 166.5), turned to 0 degrees
- moved D60 15.1 mm to (343.5, 128.7), turned to 180 degrees
Routing:
- net Net-(D15-A): track 28.0 -> 7.47 mm
- net Row3: track 322.9 -> 334.3 mm
- net Net-(D59-A): track 24.0 -> 15.7 mm
- net Row1: track 282.1 -> 288.6 mm
- net Net-(D58-A): track 13.6 -> 8.30 mm
- net Net-(D60-A): track 18.9 -> 15.6 mm
- net Net-(D87-A): track 12.2 -> 9.28 mm
- net Row4: track 320.4 -> 318.3 mm
- net Net-(D88-A): track 12.3 -> 11.1 mm
- net Row5: track 365.2 -> 364.1 mm
- net Row2: track 292.9 -> 292.1 mm
